File: xbee-usb.brd (EAGLE design)
At the start: 27 x 47 mm, 22 parts, among them U1 FT231X, U2 MCP1700, X1 ZX62D-B-5PA8

Commit message: As sent to fab.
Parts:
- removed JP2: (no value), SparkFun:1X03_LOCK
- removed X1: ZX62D-B-5PA8, zx62d-b-5pa8-oshpark_10:ZX62D-B-5PA8
- added D3: RX, _jc:D0805
- added D4: TX, _jc:D0805A
- added LOGO1: OSHW_LOGO_8MILX0100-NT, ohw-logo:OSHW_8X100_NOTEXT
- added R5, R6: 1K, _jc:M0805
- added S1: Reset, _jc:B3F-10XXOCT
- added SJ1: Reset Select, jumper:SJ_2
- moved C6 19.3 mm to (23.5, 12.0), flipped to the bottom, turned to 180 degrees
- moved L1 14.2 mm to (19.7, 11.0), flipped to the bottom, turned to 90 degrees
- moved C1 12.4 mm to (23.5, 8.80), flipped to the bottom, turned to 180 degrees
- moved JP1 5.50 mm to (19.0, 0.00)
- moved C3 5.41 mm to (11.0, 16.5), flipped to the bottom, turned to 0 degrees
- moved C2 3.04 mm to (16.0, 16.5), flipped to the bottom, turned to 180 degrees
- moved R4 3.04 mm to (8.70, 41.0)
- moved A1 3.00 mm to (13.5, 30.0)
- moved D1 3.00 mm to (23.5, 41.0)
- moved D2 3.00 mm to (3.50, 41.0)
- moved R3 3.00 mm to (17.8, 41.0)
- moved R1 2.69 mm to (15.0, 20.5), flipped to the bottom
- moved R2 2.69 mm to (12.0, 20.5), flipped to the bottom
- moved C5 1.50 mm to (20.0, 26.5), turned to 270 degrees
- moved C4 1.41 mm to (7.00, 28.5)
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Connections:
- removed net N$3: C1.1, JP1.1, L1.1
- new net +5V: C1.1, C7.1, JP1.1, L1.1, U2.3
- new net CBUS1: R5.1, U1.17
- new net CBUS2: R6.1, U1.10
- new net N$15: D4.K, R6.2
- new net N$16: S1.3, S1.4, SJ1.1
- new net N$19: SJ1.3, U1.19
- new net N$9: D3.K, R5.2
- net GND: now also S1.1, S1.2
- net N$10: now also SJ1.2
- net VCC: now also D3.A, D4.A; no longer C7.1, U2.3
Routing:
- net +5V: track 0.00 -> 43.6 mm, vias 0 -> 1
- net CBUS1: track 0.00 -> 27.2 mm, vias 0 -> 2
- net N$16: track 0.00 -> 22.5 mm
- net N$3: track 21.8 -> 0.00 mm
- net CBUS2: track 0.00 -> 19.3 mm
- net N$10: track 0.00 -> 17.0 mm
- net VCC: track 19.2 -> 30.9 mm, vias 0 -> 2
- net N$19: track 0.00 -> 11.4 mm, vias 0 -> 1
- net N$5: track 9.97 -> 6.06 mm, vias 0 -> 1
- net N$9: track 0.00 -> 2.60 mm
- net N$15: track 0.00 -> 2.60 mm
- net N$1: track 19.3 -> 17.2 mm
- net N$6: track 8.53 -> 6.91 mm, vias 0 -> 1
- net N$13: track 24.1 -> 23.0 mm, vias 0 -> 1
- net +3V3: track 10.6 -> 11.5 mm
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Other:
- board size 27 x 47 mm -> 27 x 44 mm
- board text added: "ASC"
- board text added: "BUTTON"
- board text added: "CBUS3"
- board text added: "CC BY-SA 4.0 jc 0218"
- board text added: "RESET"
- board text added: "RESET SELECT"
- board text added: "RSSI"
- board text added: "RX"
- board text added: "TX"
- board text added: "XBee USB Dongle v1.0"
- board text added: "goo.gl/xNyEkt"
- board text added: "open source"
- board text removed: "1.06in x 1.85in"
- board text removed: "27.0mm x 47.0mm"
