File: xbee-usb.sch (EAGLE design)
At the start: 22 parts, among them U1 FT231X, U2 MCP1700, X1 ZX62D-B-5PA8

Commit message: As sent to fab.
Parts:
- removed JP2: (no value), SparkFun:M03LOCK
- removed X1: ZX62D-B-5PA8, zx62d-b-5pa8-oshpark_10:ZX62D-B-5PA8
- added D3: RX, _jc:LEDD0805
- added D4: TX, _jc:LEDD0805A
- added LOGO1: OSHW_LOGO_8MILX0100-NT, ohw-logo:OSHW_LOGO_8MILX0100-NT
- added R5, R6: 1K, _jc:R-US_M0805
- added S1: Reset, _jc:10-XXOCT
- added SJ1: Reset Select, jumper:SJ2W
Connections:
- removed net N$3: C1.1, JP1.+, L1.1
- new net +5V: C1.1, C7.1, JP1.+, L1.1, U2.IN
- new net CBUS1: R5.1, U1.CBUS1
- new net CBUS2: R6.1, U1.CBUS2
- new net N$15: D4.C, R6.2
- new net N$16: S1.P, S1.P1, SJ1.1
- new net N$19: SJ1.3, U1.CBUS3
- new net N$9: D3.C, R5.2
- net GND: now also S1.S, S1.S1
- net N$10: now also SJ1.2
- net VCC: now also D3.A, D4.A; no longer C7.1, U2.IN
Other:
- moved on the sheet: A1, D1, D2, R3, R4

Commit message: Add photos, doc, BOM, etc.
Other:
- note added: "CC BY-SA"
- note added: "XBee USB Dongle by Jack Christensen is licensed under CC BY-SA 4.0 http://creativecommons.org/licenses/by-sa/4.0/"
Changed lines of the file:
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@@
 <sheet>
 <plain>
-<text x="175.26" y="30.48" size="3.81" layer="91">XBee USB Dongle</text>
+<text x="175.26" y="30.48" size="3.81" layer="91" ratio="10">XBee USB Dongle</text>
 <text x="175.26" y="25.4" size="2.54" layer="91">by Jack Christensen</text>
 <text x="264.16" y="7.62" size="2.54" layer="91">v1.0</text>
+<text x="17.78" y="22.86" size="3.81" layer="91" ratio="10">CC BY-SA</text>
+<text x="17.78" y="15.24" size="2.1844" layer="91" ratio="10">XBee USB Dongle by Jack Christensen is licensed
+under CC BY-SA 4.0 http://creativecommons.org/licenses/by-sa/4.0/</text>
 </plain>
 <instances>
@@
 <instance part="P+5" gate="1" x="48.26" y="154.94"/>
 <instance part="P+4" gate="1" x="96.52" y="96.52"/>
-<instance part="LOGO1" gate="G$1" x="165.1" y="33.02"/>
+<instance part="LOGO1" gate="G$1" x="53.34" y="25.4"/>
 <instance part="S1" gate="1" x="160.02" y="121.92" smashed="yes" rot="R180">
 <attribute name="NAME" x="149.86" y="118.11" size="1.778" layer="95"/>
@@
 </schematic>
 </drawing>
+<compatibility>
+<note version="6.3" minversion="6.2.2" severity="warning">
+Since Version 6.2.2 text objects can contain more than one line,
+which will not be processed correctly with this version.
+</note>
+</compatibility>
 </eagle>
